File: pixel_pi_hat.sch (KiCad schematic (older format))
At the start: 8 parts, among them J1 Conn_01x02_Male, J2 Conn_01x03_Male, J3 Conn_02x20_Odd_Even, U1 74125

Commit message: Change to wago 804 push button terminals
Parts:
- added J4: Conn_01x02_Male, Connector_PinHeader_2.54mm:PinHeader_1x02_P2.54mm_Vertical, symbol Connector:Conn_01x02_Male
- J1: footprint Connector_PinHeader_2.54mm:PinHeader_1x02_P2.54mm_Vertical -> TerminalBlock_WAGO:TerminalBlock_WAGO_804-102_1x02_P5.00mm_45Degree
- J2: footprint Connector_PinHeader_2.54mm:PinHeader_1x03_P2.54mm_Vertical -> TerminalBlock_WAGO:TerminalBlock_WAGO_804-103_1x03_P5.00mm_45Degree
Connections:
- net +5V: now also J4.2 (Pin_2); no longer J3.2 (Pin_2), J3.4 (Pin_4)
- new net: J3.2 (Pin_2), J3.4 (Pin_4), J4.1 (Pin_1)
Changed lines of the file:
@@
 F 0 "J1" H 3603 1606 50  0000 C CNN
 F 1 "Conn_01x02_Male" H 3603 1515 50  0000 C CNN
-F 2 "Connector_PinHeader_2.54mm:PinHeader_1x02_P2.54mm_Vertical" H 3495 1425 50  0001 C CNN
+F 2 "TerminalBlock_WAGO:TerminalBlock_WAGO_804-102_1x02_P5.00mm_45Degree" H 3495 1425 50  0001 C CNN
 F 3 "~" H 3495 1425 50  0001 C CNN
 	1    3495 1425
@@
 F 0 "J2" H 3603 2211 50  0000 C CNN
 F 1 "Conn_01x03_Male" H 3603 2120 50  0000 C CNN
-F 2 "Connector_PinHeader_2.54mm:PinHeader_1x03_P2.54mm_Vertical" H 3495 1930 50  0001 C CNN
+F 2 "TerminalBlock_WAGO:TerminalBlock_WAGO_804-103_1x03_P5.00mm_45Degree" H 3495 1930 50  0001 C CNN
 F 3 "~" H 3495 1930 50  0001 C CNN
 	1    3495 1930
@@
 	6680 1645 6585 1645
 Wire Wire Line
-	4835 1145 6765 1145
+	4835 1145 5660 1145
 Wire Wire Line
 	6765 1145 6765 1590
@@
 Wire Wire Line
 	4555 2030 4835 2030
+$Comp
+L Connector:Conn_01x02_Male J4
+U 1 1 615ED83F
+P 5760 945
+F 0 "J4" V 5822 989 50  0000 L CNN
+F 1 "Conn_01x02_Male" V 5913 989 50  0000 L CNN
+F 2 "Connector_PinHeader_2.54mm:PinHeader_1x02_P2.54mm_Vertical" H 5760 945 50  0001 C CNN
+F 3 "~" H 5760 945 50  0001 C CNN
+	1    5760 945
+	0    1    1    0
+$EndComp
+Wire Wire Line
+	5760 1145 6765 1145
 $EndSCHEMATC
